Commit message: Migrate reviewed Revo3 right-hand convex collisions into URDF

File: revo3_system/urdf/revo3_right.urdf (robot description, URDF)
Before this commit: robot revo3_single, 58 links, 57 joints
Links:
- link right_hand_base_link: geometry visual mesh filename=../meshes/hands/visual/right/right_hand_base_link.STL
- link right_index_DIP_link: geometry collision mesh filename=../meshes/hands/collision/right/optimized_20261027/DIP/revo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; collision mesh filename=../meshes/hands/collision/right/optimized_20261027/DIP/revo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
- link right_index_DIP_rubber_link: geometry visual mesh filename=../meshes/hands/visual/right/right_index_DIP_rubber_link.STL
- link right_index_MCP_link: geometry collision mesh filename=../meshes/hands/collision/right/optimized_20261027/MCP/revo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; collision mesh filename=../meshes/hands/collision/right/optimized_20261027/MCP/revo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
- link right_index_MCP_rubber_link: geometry visual mesh filename=../meshes/hands/visual/right/right_index_MCP_rubber_link.STL
- link right_index_MCP_touch_link: geometry visual mesh filename=../meshes/hands/visual/right/right_index_MCP_touch_link.STL
- link right_index_MPR_link: geometry collision mesh filename=../meshes/hands/collision/right/optimized_20261027/MPR_side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; collision mesh filename=../meshes/hands/collision/right/optimized_20261027/MPR_side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
- link right_index_PIP_link: geometry collision mesh filename=../meshes/hands/collision/right/optimized_20261027/PIP/revo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; collision mesh filename=../meshes/hands/collision/right/optimized_20261027/PIP/revo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
- link right_index_PIP_rubber_link: geometry visual mesh filename=../meshes/hands/visual/right/right_index_PIP_rubber_link.STL
- link right_index_PIP_touch_link: geometry visual mesh filename=../meshes/hands/visual/right/right_index_PIP_touch_link.STL
- link right_little_DIP_link: geometry collision mesh filename=../meshes/hands/collision/right/optimized_20261027/DIP/revo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; collision mesh filename=../meshes/hands/collision/right/optimized_20261027/DIP/revo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
- link right_little_DIP_rubber_link: geometry visual mesh filename=../meshes/hands/visual/right/right_little_DIP_rubber_link.S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
- link right_little_MCP_link: geometry collision mesh filename=../meshes/hands/collision/right/optimized_20261027/MCP/revo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; collision mesh filename=../meshes/hands/collision/right/optimized_20261027/MCP/revo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
- link right_little_MCP_rubber_link: geometry visual mesh filename=../meshes/hands/visual/right/right_little_MCP_rubber_link.S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
- link right_little_MCP_touch_link: geometry visual mesh filename=../meshes/hands/visual/right/right_little_MCP_touch_link.STL
- link right_little_MPR_link: geometry collision mesh filename=../meshes/hands/collision/right/optimized_20261027/MPR_side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; collision mesh filename=../meshes/hands/collision/right/optimized_20261027/MPR_side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
- link right_little_PIP_link: geometry collision mesh filename=../meshes/hands/collision/right/optimized_20261027/PIP/revo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; collision mesh filename=../meshes/hands/collision/right/optimized_20261027/PIP/revo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
- link right_little_PIP_rubber_link: geometry visual mesh filename=../meshes/hands/visual/right/right_little_PIP_rubber_link.S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
- link right_little_PIP_touch_link: geometry visual mesh filename=../meshes/hands/visual/right/right_little_PIP_touch_link.STL
- link right_middle_DIP_link: geometry collision mesh filename=../meshes/hands/collision/right/optimized_20261027/DIP/revo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; collision mesh filename=../meshes/hands/collision/right/optimized_20261027/DIP/revo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
- link right_middle_DIP_rubber_link: geometry visual mesh filename=../meshes/hands/visual/right/right_middle_DIP_rubber_link.S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
- link right_middle_MCP_link: geometry collision mesh filename=../meshes/hands/collision/right/optimized_20261027/MCP/revo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; collision mesh filename=../meshes/hands/collision/right/optimized_20261027/MCP/revo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
- link right_middle_MCP_rubber_link: geometry visual mesh filename=../meshes/hands/visual/right/right_middle_MCP_rubber_link.S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
- link right_middle_MCP_touch_link: geometry visual mesh filename=../meshes/hands/visual/right/right_middle_MCP_touch_link.STL
- link right_middle_MPR_link: geometry collision mesh filename=../meshes/hands/collision/right/optimized_20261027/MPR_side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; collision mesh filename=../meshes/hands/collision/right/optimized_20261027/MPR_side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
- link right_middle_PIP_link: geometry collision mesh filename=../meshes/hands/collision/right/optimized_20261027/PIP/revo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; collision mesh filename=../meshes/hands/collision/right/optimized_20261027/PIP/revo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
- link right_middle_PIP_rubber_link: geometry visual mesh filename=../meshes/hands/visual/right/right_middle_PIP_rubber_link.S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
- link right_middle_PIP_touch_link: geometry visual mesh filename=../meshes/hands/visual/right/right_middle_PIP_touch_link.STL
- link right_palm_led_link: geometry visual mesh filename=../meshes/hands/visual/right/right_palm_led_link.dae
- link right_palm_link: geometry visual mesh filename=../meshes/hands/visual/right/right_palm_link__revo3_aluminu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; visual mesh filename=../meshes/hands/visual/right/right_palm_link__revo3_white_p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
- link right_palm_rubber_link: geometry collision mesh filename=../meshes/hands/collision/right/optimized_20261027/right_pa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; collision mesh filename=../meshes/hands/collision/right/optimized_20261027/right_pa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
- link right_palm_touch_link: geometry visual mesh filename=../meshes/hands/visual/right/right_palm_touch_link.STL
- link right_ring_DIP_link: geometry collision mesh filename=../meshes/hands/collision/right/optimized_20261027/DIP/revo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; collision mesh filename=../meshes/hands/collision/right/optimized_20261027/DIP/revo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
- link right_ring_DIP_rubber_link: geometry visual mesh filename=../meshes/hands/visual/right/right_ring_DIP_rubber_link.STL
- link right_ring_MCP_link: geometry collision mesh filename=../meshes/hands/collision/right/optimized_20261027/MCP/revo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; collision mesh filename=../meshes/hands/collision/right/optimized_20261027/MCP/revo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
- link right_ring_MCP_rubber_link: geometry visual mesh filename=../meshes/hands/visual/right/right_ring_MCP_rubber_link.STL
- link right_ring_MCP_touch_link: geometry visual mesh filename=../meshes/hands/visual/right/right_ring_MCP_touch_link.STL
- link right_ring_MPR_link: geometry collision mesh filename=../meshes/hands/collision/right/optimized_20261027/MPR_side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; collision mesh filename=../meshes/hands/collision/right/optimized_20261027/MPR_side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
- link right_ring_PIP_link: geometry collision mesh filename=../meshes/hands/collision/right/optimized_20261027/PIP/revo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; collision mesh filename=../meshes/hands/collision/right/optimized_20261027/PIP/revo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
- link right_ring_PIP_rubber_link: geometry visual mesh filename=../meshes/hands/visual/right/right_ring_PIP_rubber_link.STL
- link right_ring_PIP_touch_link: geometry visual mesh filename=../meshes/hands/visual/right/right_ring_PIP_touch_link.STL
- link right_thumb_CMP_link: geometry collision mesh filename=../meshes/hands/collision/right/optimized_20261027/right_th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; collision mesh filename=../meshes/hands/collision/right/optimized_20261027/right_th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
- link right_thumb_CMR_link: geometry collision mesh filename=../meshes/hands/collision/right/optimized_20261027/right_th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; collision mesh filename=../meshes/hands/collision/right/optimized_20261027/right_th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
- link right_thumb_DIP_link: geometry collision mesh filename=../meshes/hands/collision/right/optimized_20261027/right_th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; collision mesh filename=../meshes/hands/collision/right/optimized_20261027/right_th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
- link right_thumb_DIP_rubber_link: geometry visual mesh filename=../meshes/hands/visual/right/right_thumb_DIP_rubber_link.STL
- link right_thumb_MCP_link: geometry collision mesh filename=../meshes/hands/collision/right/optimized_20261027/right_th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; collision mesh filename=../meshes/hands/collision/right/optimized_20261027/right_th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
- link right_thumb_MCP_rubber_link: geometry visual mesh filename=../meshes/hands/visual/right/right_thumb_MCP_rubber_link.STL
- link right_thumb_MCP_touch_link: geometry visual mesh filename=../meshes/hands/visual/right/right_thumb_MCP_touch_link.STL
- link right_thumb_PIP_link: geometry collision mesh filename=../meshes/hands/collision/right/optimized_20261027/right_th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; collision mesh filename=../meshes/hands/collision/right/optimized_20261027/right_th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
- link right_thumb_PIP_rubber_link: geometry visual mesh filename=../meshes/hands/visual/right/right_thumb_PIP_rubber_link.STL
- link right_thumb_PIP_touch_link: geometry visual mesh filename=../meshes/hands/visual/right/right_thumb_PIP_touch_link.STL
